File: board/the-intercept/the-intercept.kicad_pcb (KiCad board)
At the start: 2 copper layers, 63.5 x 45.7 mm, 35 parts, among them J1 USB_B_Micro, Q1 Q_Photo_NPN, SW1 SW_Push, SW2 SW_Push, U1 ESP32-WROOM-32D, U2 93LCxxB, U3 FT232H, U4 LM1117-3.3, Y1 12MHz

Commit message: Revision two of the board
Parts:
- U2: footprint Package_SO:SOIC-8-1EP_3.9x4.9mm_P1.27mm_EP2.29x3mm -> Package_SO:SOIC-8_3.9x4.9mm_P1.27mm
- U3: footprint Package_QFP:LQFP-48-1EP_7x7mm_P0.5mm_EP3.6x3.6mm -> Package_QFP:LQFP-48_7x7mm_P0.5mm
- Y1: value 12MHz -> Crystal_GND24_Small
- moved C4 4.52 mm to (161.8, 115.6), turned to 0 degrees
- moved C6 4.34 mm to (165.1, 112.8), turned to 270 degrees
- moved R9 1.27 mm to (144.8, 109.5), turned to 0 degrees
- moved D1 1.27 mm to (169.5, 115.6)
- moved C3 0.98 mm to (146.8, 112.4), turned to 180 degrees
- moved R2 0.79 mm to (152.7, 89.9)
- moved R10 0.74 mm to (144.8, 107.9), turned to 0 degrees
- moved R7 0.64 mm to (147.4, 121.4)
- moved C9 0.28 mm to (154.7, 113.8)
- moved Y1 0.12 mm to (161.8, 112.8), turned to 0 degrees
Connections:
- Y1 pad 2: Net-(C6-Pad1) -> GND
- Y1 pad 3: (no net) -> Net-(C6-Pad1)
- Y1 pad 4: (no net) -> GND
Routing:
- net GND: track 243.9 -> 121.4 mm, vias 5 -> 16
- net VCCIO: track 179.4 -> 164.3 mm, vias 8 -> 0
- net VBUS: track 41.6 -> 35.7 mm
- net Net-(C4-Pad1): track 13.9 -> 8.39 mm
- net Net-(C6-Pad1): track 7.94 -> 10.5 mm
- net Net-(R9-Pad2): track 3.95 -> 1.85 mm
- net left_lever: track 26.2 -> 25.5 mm
- net DATA: track 14.6 -> 13.9 mm
- net Net-(R7-Pad1): track 2.92 -> 2.27 mm

Commit message: Updates for final board
Parts:
- moved R3 7.56 mm to (153.8, 129.5), turned to 180 degrees
- moved R2 1.69 mm to (154.2, 89.2), turned to 180 degrees
- turned SW2 to 180 degrees
Routing:
- net GND: track 121.4 -> 113.4 mm, vias 16 -> 17
- net VCCIO: track 164.3 -> 158.8 mm
- net right_lever: track 25.6 -> 30.9 mm
- net left_lever: track 25.5 -> 26.3 mm
